File: HW/HDMI-LVDS.brd (EAGLE design)
At the start: 88.4 x 52.2 mm, 112 parts, among them IC1 TFP401A-PAD, IC2 24LC02B, IC3 IS31BL3506A-TTLS2, IC4 ATMEGA32U4-MU, IC5 LDO-TS1117CW-3V3, J1 DCJ0202, J20_1 JUMPER2-0402, J20_2 JUMPER2-0402, J30_1 JUMPER2-0402, J30_2 JUMPER2-0402, Q1 16MHz, SW1 SW-TACTILE-PTS840P, T6 BSS138PS, T7 BSS138PS, T8 BSS138PS, U1 SN75LVDS83BDGG, X1 PASSER-07, X2 PASSER-07, X3 PASSER-07, X4 PASSER-07

Commit message: last version
Parts:
- removed SJ1: (no value), jumper:SJ
- removed TP_BOT: FPC04, we-con:FPC04
- added C25, C26, C27, C28: 10n, we-rcl:C0402
- added SV3, SV5: (no value), con-lsta:FE08
- added SV4: (no value), con-lstb:MA04-2
- added SV6: (no value), con-lsta:FE06
- SV2: device con-lstb:MA04-1 -> con-lsta:FE10
- moved J1 88.1 mm to (-29.5, 25.6), flipped to the top
- moved SV2 79.5 mm to (-24.5, 49.7)
- moved USB 23.3 mm to (56.4, 0.20), turned to 270 degrees
- moved X1 17.1 mm to (18.8, -9.29)
- moved X2 14.7 mm to (2.42, 61.3)
- moved R17 12.7 mm to (57.9, 5.71), turned to 180 degrees
- moved R19 11.7 mm to (50.3, 27.8)
- moved LED2 11.7 mm to (53.1, 27.8)
- moved R18 11.5 mm to (50.3, 26.0)
- moved LED1 11.5 mm to (53.1, 26.0)
- moved JP1 10.6 mm to (51.7, 5.80), turned to 0 degrees
- moved R11 9.60 mm to (11.5, 40.6), turned to 270 degrees
- moved R5 9.10 mm to (11.5, 45.7), turned to 90 degrees
- moved R8 8.95 mm to (11.5, 41.9), turned to 270 degrees
- moved R7 8.69 mm to (11.5, 44.4), turned to 90 degrees
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Connections:
- removed net PI+: SJ1.1
- net +3V3: now also C25.2, C26.2, C27.2, C28.2; no longer U1.30
- net +5V: now also SV4.6, SV4.8; no longer SJ1.2, SV2.3, SV2.4
- net DE: now also U1.30
- net GND: now also C25.1, C26.1, C27.1, C28.1, SV4.2, SV4.4; no longer SV2.1, SV2.2
- net X+: now also SV4.7; no longer TP_BOT.4
- net X-: now also SV4.5; no longer TP_BOT.2
- net Y+: now also SV4.3; no longer TP_BOT.1
- net Y-: now also SV4.1; no longer TP_BOT.3
Routing:
- net N$10: track 14.0 -> 113.3 mm, vias 0 -> 1
- net X-: track 78.3 -> 17.2 mm
- net PWM3: track 42.4 -> 0.00 mm, vias 4 -> 1
- net Y-: track 77.1 -> 40.7 mm, vias 4 -> 3
- net Y+: track 72.6 -> 37.1 mm, vias 3 -> 2
- net X+: track 79.3 -> 48.3 mm
- net DE: track 32.1 -> 52.7 mm
- net USBD_P: track 19.4 -> 37.1 mm
- net USBD_N: track 19.1 -> 35.9 mm
- net LV_PWM2: track 34.3 -> 18.6 mm
- net LED2: track 12.1 -> 27.2 mm, vias 2 -> 4
- net LED1: track 12.6 -> 27.2 mm, vias 2 -> 4
- net +5V: track 198.8 -> 209.4 mm
- net USBV: track 10.8 -> 3.07 mm, vias 0 -> 2
- net STAG: track 11.9 -> 5.58 mm
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Other:
- board size 88.4 x 52.2 mm -> 99.9 x 54.6 mm
- board text removed: "HDMI-Display Rev 1.1"
- board text removed: "github.com/watterott/HDMI-Display"
- board text removed: "watterott.com"
