File: HW/HDMI-LVDS.sch (EAGLE design)
At the start: 112 parts, among them IC1 TFP401A-PAD, IC2 24LC02B, IC3 IS31BL3506A-TTLS2, IC4 ATMEGA32U4-MU, IC5 LDO-TS1117CW-3V3, J1 DCJ0202, J20_1 JUMPER2-0402, J20_2 JUMPER2-0402, J30_1 JUMPER2-0402, J30_2 JUMPER2-0402, Q1 16MHz, SW1 SW-TACTILE-PTS840P, T6 BSS138PS, T7 BSS138PS, T8 BSS138PS, U1 SN75LVDS83BDGG, X1 PASSER-07, X2 PASSER-07, X3 PASSER-07, X4 PASSER-07

Commit message: last version
Parts:
- removed SJ1: (no value), jumper:SJ
- removed TP_BOT: FPC04, we-con:FPC04
- added C25, C26, C27, C28: 10n, we-rcl:CAPACITOR-0402
- added SV3, SV5: (no value), con-lsta:FE08-1
- added SV4: (no value), con-lstb:MA04-2
- added SV6: (no value), con-lsta:FE06-1
- SV2: device con-lstb:MA04-1 -> con-lsta:FE10-1
Connections:
- removed net PI+: SJ1.1
- net +3V3: now also C25.2, C26.2, C27.2, C28.2; no longer U1.D26
- net +5V: now also SV4.6, SV4.8; no longer SJ1.2, SV2.3, SV2.4
- net DE: now also U1.D26
- net GND: now also C25.1, C26.1, C27.1, C28.1, SV4.2, SV4.4; no longer SV2.1, SV2.2
- net X+: now also SV4.7; no longer TP_BOT.4
- net X-: now also SV4.5; no longer TP_BOT.2
- net Y+: now also SV4.3; no longer TP_BOT.1
- net Y-: now also SV4.1; no longer TP_BOT.3
